File: little_clock/little_clock.sch (KiCad schematic (older format))
At the start: 37 parts

Commit message: little_clock sch Ver.1.0
little_clock sch Ver.1.0
Parts:
- C3, C4: renamed from C?; value C -> 0.1uF
- DS1: renamed from DS?; footprint RC1602A -> Display:RC1602A
- L1: renamed from L?; value L -> 30uH
- R1: renamed from R?; value R -> 10K
- R2: renamed from R?; value R -> 1K
- R3: renamed from R?; value R -> 220
- gave numbers to parts that had none: 30
Connections:
- net BL: now also IC1.16 ((PCINT2/OC1B/~SS~)PB2)
- net BUZZ_control: now also IC1.17 ((PCINT3/OC2A/MOSI)PB3)
- net Back/Alarm: now also IC1.4 ((PCINT18/INT0)PD2)
- net DHT11_DATA: now also IC1.23 ((PCINT8/ADC0)PC0)
- net LCM_D4: now also IC1.12 ((PCINT22/OC0A/AIN0)PD6)
- net LCM_D5: now also IC1.13 ((PCINT23/AIN1)PD7)
- net LCM_D6: now also IC1.14 ((PCINT0/CLKO/ICP1)PB0)
- net LCM_D7: now also IC1.15 ((PCINT1/OC1A)PB1)
- net LCM_E: now also IC1.11 ((PCINT21/OC0B/T1)PD5)
- net LCM_RS: now also IC1.6 ((PCINT20/XCK/T0)PD4)
- net Menu/Enter: now also IC1.26 ((PCINT11/ADC3)PC3)
- net Vo: now also IC1.5 ((PCINT19/OC2B/INT1)PD3)
- net func_DOWN: now also IC1.25 ((PCINT10/ADC2)PC2)
- net func_UP: now also IC1.24 ((PCINT9/ADC1)PC1)
