File: little_clock/little_clock.sch (KiCad schematic (older format))
At the start: 38 parts, among them CON1 BARREL_JACK, IC1 ATMEGA328-P, P1 DS1307_BAT, P2 DHT11, Q1 2N2222, Q2 2N2222, SW1 UP_button, SW2 DOWN_button, SW3 B/A_button, SW4 M/E_button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

Commit message: design Ver1.2
design Ver1.2
Parts:
- added C13: 0.1u, Capacitors_SMD:C_1812_HandSoldering, symbol C
- added P3, P4: POWER_CONN, Pin_Headers:Pin_Header_Straight_2x01_Pitch2.54mm, symbol CONN_01X02
- added P5, P6: CONN_01X05, Pin_Headers:Pin_Header_Straight_1x05_Pitch2.54mm, symbol CONN_01X05
- C1: footprint Capacitors_SMD:CP_Elec_4x5.7 -> Capacitors_Tantalum_SMD:CP_Tantalum_Case-D_EIA-7343-31_Wave
- C10, C3, C4, C6, C7, C8, C9: footprint Capacitors_SMD:C_1210_HandSoldering -> Capacitors_SMD:C_1812_HandSoldering
- C2: footprint Capacitors_SMD:C_1210_HandSoldering -> Capacitors_Tantalum_SMD:CP_Tantalum_Case-X_EIA-7343-43_Wave
- Q1, Q2: footprint TO_SOT_Packages_SMD:TO-252-2Lead -> TO_SOT_Packages_SMD:SOT89-3_Housing_Handsoldering
Connections:
- net 5V_POWER: now also P4.1 (P1); no longer BZ1.1 (-), C2.2, DS1.2 (VDD), IC1.7 (VCC), L1.1, R1.1, R3.1, R6.1, RN1.1 (common)
- net BUZZ_control: now also P5.2 (P2); no longer IC1.17 ((PCINT3/OC2A/MOSI)PB3)
- net DHT11_DATA: now also P5.5 (P5); no longer IC1.23 ((PCINT8/ADC0)PC0)
- net DS1307_SCL: now also P5.3 (P3); no longer IC1.28 ((PCINT13/SCL/ADC5)PC5)
- net DS1307_SDA: now also P5.4 (P4); no longer IC1.27 ((PCINT12/SDA/ADC4)PC4)
- net GND: now also C13.2, P3.2 (P2), P6.5 (P5); no longer C10.2, C5.2, C6.2, C8.1, C9.2, CON1.2, CON1.3, P1.1 (P1), P2.4 (P4), U1.4 (GND)
- new net: IC1.17 ((PCINT3/OC2A/MOSI)PB3), P6.1 (P1)
- new net: IC1.23 ((PCINT8/ADC0)PC0), P6.2 (P2)
- new net: IC1.27 ((PCINT12/SDA/ADC4)PC4), P6.3 (P3)
- new net: IC1.28 ((PCINT13/SCL/ADC5)PC5), P6.4 (P4)
- new net G: C10.2, C5.2, C6.2, C8.1, C9.2, CON1.2, CON1.3, P1.1 (P1), P2.4 (P4), P4.2 (P2), P5.1 (P1), U1.4 (GND)
- new net conn_VCC: BZ1.1 (-), C13.1, C2.2, DS1.2 (VDD), IC1.7 (VCC), L1.1, P3.1 (P1), R1.1, R3.1, R6.1, RN1.1 (common)

Commit message: PCB Design Ver.1.0Beta
PCB Design Ver.1.0Beta
Parts:
- removed C13: 0.1u, Capacitors_SMD:C_1812_HandSoldering, symbol C
- removed DS1: RC1602A-GHW-ESX, Pin_Headers:Pin_Header_Straight_1x16_Pitch2.54mm, symbol RC1602A-GHW-ESX
- removed P3, P4: POWER_CONN, Pin_Headers:Pin_Header_Straight_2x01_Pitch2.54mm, symbol CONN_01X02
- removed P6: CONN_01X05, Pin_Headers:Pin_Header_Straight_1x05_Pitch2.54mm, symbol CONN_01X05
- removed RN1: 10K, Pin_Headers:Pin_Header_Straight_1x05_Pitch2.54mm, symbol R_Network04
- added P10: DHT11_conn_B, Pin_Headers:Pin_Header_Straight_1x04_Pitch2.54mm, symbol CONN_01X04
- added P11: DHT11_conn_A, Pin_Headers:Pin_Header_Straight_1x04_Pitch2.54mm, symbol CONN_01X04
- added P4: SW_Part_B, Pin_Headers:Pin_Header_Straight_1x05_Pitch2.54mm, symbol CONN_01X05
- added P6: LCM_P, Pin_Headers:Pin_Header_Straight_1x06_Pitch2.54mm, symbol CONN_01X06
- added P7: LCM_D, Pin_Headers:Pin_Header_Straight_1x06_Pitch2.54mm, symbol CONN_01X06
- added P8: DS1307_conn_A, Pin_Headers:Pin_Header_Straight_1x04_Pitch2.54mm, symbol CONN_01X04
- added P9: DS1307_conn_B, Pin_Headers:Pin_Header_Straight_1x04_Pitch2.54mm, symbol CONN_01X04
- added R10, R11, R12, R9: 10k, Resistors_ThroughHole:R_Axial_DIN0207_L6.3mm_D2.5mm_P10.16mm_Horizontal, symbol R
- C1: footprint Capacitors_Tantalum_SMD:CP_Tantalum_Case-D_EIA-7343-31_Wave -> Capacitors_ThroughHole:CP_Radial_D5.0mm_P2.50mm
- C10, C6, C7, C8, C9: footprint Capacitors_SMD:C_1812_HandSoldering -> Capacitors_ThroughHole:C_Disc_D5.0mm_W2.5mm_P5.00mm
- C11, C12: footprint Capacitors_SMD:C_0805_HandSoldering -> Capacitors_ThroughHole:C_Disc_D3.0mm_W1.6mm_P2.50mm
- C2: footprint Capacitors_Tantalum_SMD:CP_Tantalum_Case-X_EIA-7343-43_Wave -> Capacitors_ThroughHole:C_Disc_D5.0mm_W2.5mm_P5.00mm
- C3, C4: footprint Capacitors_SMD:C_1812_HandSoldering -> Capacitors_ThroughHole:C_Disc_D4.7mm_W2.5mm_P5.00mm
- C5: footprint Capacitors_SMD:CP_Elec_4x5.7 -> Capacitors_ThroughHole:CP_Radial_D5.0mm_P2.50mm
- P1: footprint Sockets_WAGO734:WAGO_734_2pin_Straight_RuggedPads -> Socket_Strips:Socket_Strip_Straight_2x01_Pitch2.54mm
- P5: value CONN_01X05 -> SW_Part_A
- Q1, Q2: footprint TO_SOT_Packages_SMD:SOT89-3_Housing_Handsoldering -> TO_SOT_Packages_THT:TO-92_Inline_Wide
- SW1, SW2, SW3, SW4: footprint Buttons_Switches_ThroughHole:SW_Tactile_SKHH_Angled -> Buttons_Switches_ThroughHole:SW_PUSH_SMALL
Connections:
- net conn_VCC is gone; now on net 5V_POWER: BZ1.1 (-), C2.2, IC1.7 (VCC), L1.1, R1.1, R3.1, R6.1
- net 5V_POWER: now also P10.1 (P1), P6.2 (P2), P9.1 (P1), R10.2, R11.2, R12.2, R9.2; no longer C10.1, C9.1, P2.1 (P1), R4.2, R7.1, R8.1, U1.8 (VCC)
- net BL: now also IC1.15 ((PCINT1/OC1A)PB1); no longer IC1.16 ((PCINT2/OC1B/~SS~)PB2)
- net BUZZ_control: now also IC1.17 ((PCINT3/OC2A/MOSI)PB3); no longer P5.2 (P2)
- net Back/Alarm: now also IC1.26 ((PCINT11/ADC3)PC3), P5.1 (P1); no longer IC1.4 ((PCINT18/INT0)PD2), SW3.1
- net DHT11_DATA: now also P11.3 (P3); no longer P5.5 (P5)
- net DS1307_SCL: now also P8.3 (P3); no longer P5.3 (P3)
- net DS1307_SDA: now also P8.2 (P2); no longer P5.4 (P4)
- net GND: now also C5.2, C6.2, CON1.2, CON1.3, P5.5 (P5), P10.4 (P4), P6.1 (P1), P6.5 (P5), P7.6 (P6), P9.4 (P4); no longer SW1.2, SW2.2, SW3.2, SW4.2
- net LCM_D4: now also IC1.11 ((PCINT21/OC0B/T1)PD5), P7.1 (P1), R9.1; no longer IC1.12 ((PCINT22/OC0A/AIN0)PD6)
- net LCM_D5: now also IC1.12 ((PCINT22/OC0A/AIN0)PD6), P7.2 (P2), R10.1; no longer IC1.13 ((PCINT23/AIN1)PD7)
- net LCM_D6: now also IC1.13 ((PCINT23/AIN1)PD7), P7.3 (P3), R11.1; no longer IC1.14 ((PCINT0/CLKO/ICP1)PB0)
- net LCM_D7: now also IC1.14 ((PCINT0/CLKO/ICP1)PB0), P7.4 (P4), R12.1; no longer IC1.15 ((PCINT1/OC1A)PB1)
- net LCM_E: now also IC1.6 ((PCINT20/XCK/T0)PD4), P6.6 (P6); no longer IC1.11 ((PCINT21/OC0B/T1)PD5)
- net LCM_RS: now also IC1.5 ((PCINT19/OC2B/INT1)PD3), P6.4 (P4); no longer IC1.6 ((PCINT20/XCK/T0)PD4)
- net Menu/Enter: now also IC1.24 ((PCINT9/ADC1)PC1), P5.3 (P3); no longer IC1.26 ((PCINT11/ADC3)PC3), SW4.1
- net Vo: now also IC1.4 ((PCINT18/INT0)PD2), P6.3 (P3); no longer IC1.5 ((PCINT19/OC2B/INT1)PD3)
- net func_DOWN: now also IC1.23 ((PCINT8/ADC0)PC0), P5.4 (P4); no longer IC1.25 ((PCINT10/ADC2)PC2), SW2.1
- net func_UP: now also IC1.25 ((PCINT10/ADC2)PC2), P5.2 (P2); no longer IC1.24 ((PCINT9/ADC1)PC1), SW1.1
- net at IC1.27 ((PCINT12/SDA/ADC4)PC4): now also P9.2 (P2)
- net at IC1.28 ((PCINT13/SCL/ADC5)PC5): now also P9.3 (P3)
- net at Q1.1 (E): now also P7.5 (P5)
- net at C8.2, U1.3 (VBATT): now also P1.1 (P1); no longer P1.2 (P2)
- removed net G: C10.2, C5.2, C6.2, C8.1, C9.2, CON1.2, CON1.3, P1.1 (P1), P2.4 (P4), P5.1 (P1), U1.4 (GND)
- new net: IC1.16 ((PCINT2/OC1B/~SS~)PB2), P10.3 (P3)
- new net: P4.5 (P5), SW1.1, SW2.2, SW3.2, SW4.2
- new net: P4.2 (P2), SW1.2
- new net: P4.4 (P4), SW2.1
- new net: P4.1 (P1), SW3.1
- new net: P4.3 (P3), SW4.1
- new net DHT11_Power: C10.1, P11.1 (P1), P2.1 (P1), R4.2
- new net DS1307_Power: C9.1, P8.1 (P1), R7.1, R8.1, U1.8 (VCC)
- new net G1: C8.1, C9.2, P1.2 (P2), P8.4 (P4), U1.4 (GND)
- new net G2: C10.2, P11.4 (P4), P2.4 (P4)
Other:
- moved on the sheet: SW1, SW2, SW3, SW4
