File: little_clock/little_clock.kicad_pcb (KiCad board)
At the start: 2 copper layers, 38 parts, among them CON1 BARREL_JACK, IC1 ATMEGA328-P, P1 DS1307_BAT, P2 DHT11, Q1 2N2222, Q2 2N2222, SW1 UP_button, SW2 DOWN_button, SW3 B/A_button, SW4 M/E_button, U1 DS1307, Y1 32.768KHz, Y2 16MHz

Commit message: design Ver1.2
design Ver1.2
Parts:
- added C13: 0.1u, Capacitors_SMD:C_1812_HandSoldering, F.Cu at (267.0, 56.0)
- added P3: POWER_CONN, Pin_Headers:Pin_Header_Straight_2x01_Pitch2.54mm, F.Cu at (268.0, 60.0)
- added P4: POWER_CONN, Pin_Headers:Pin_Header_Straight_2x01_Pitch2.54mm, F.Cu at (160.0, 76.0)
- added P5: CONN_01X05, Pin_Headers:Pin_Header_Straight_1x05_Pitch2.54mm, F.Cu at (184.0, 46.0)
- added P6: CONN_01X05, Pin_Headers:Pin_Header_Straight_1x05_Pitch2.54mm, F.Cu at (213.0, 39.0)
- C1: footprint Capacitors_SMD:CP_Elec_4x5.7 -> Capacitors_Tantalum_SMD:CP_Tantalum_Case-D_EIA-7343-31_Wave
- C10, C3, C4, C6, C7, C8, C9: footprint Capacitors_SMD:C_1210_HandSoldering -> Capacitors_SMD:C_1812_HandSoldering
- C2: footprint Capacitors_SMD:C_1210_HandSoldering -> Capacitors_Tantalum_SMD:CP_Tantalum_Case-X_EIA-7343-43_Wave
- Q1, Q2: footprint TO_SOT_Packages_SMD:TO-252-2Lead -> TO_SOT_Packages_SMD:SOT89-3_Housing_Handsoldering
- moved SW3 197.6 mm to (271.0, 31.0)
- moved SW4 171.5 mm to (258.0, 31.0)
- moved L1 156.1 mm to (248.0, 39.0), turned to 180 degrees
- moved BZ1 148.1 mm to (271.0, 43.0), turned to 270 degrees
- moved C4 144.6 mm to (232.0, 39.0)
- moved SW2 143.7 mm to (201.0, 47.0)
- moved SW1 143.4 mm to (201.0, 36.0)
- moved C12 129.3 mm to (243.0, 59.0), turned to 0 degrees
- moved Y2 126.6 mm to (237.0, 55.0), turned to 0 degrees
- moved R1 121.6 mm to (231.0, 54.0), turned to 180 degrees
- moved C11 121.6 mm to (236.0, 59.0), turned to 0 degrees
- moved R3 117.1 mm to (248.0, 37.0), turned to 180 degrees
- moved D1 116.9 mm to (268.0, 52.0)
- moved P2 114.6 mm to (171.0, 114.0)
- moved C3 106.6 mm to (215.0, 54.0), turned to 180 degrees
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Connections:
- BZ1 pad 1: 5V_POWER -> conn_VCC
- C10 pad 2: GND -> G
- C2 pad 2: 5V_POWER -> conn_VCC
- C5 pad 2: GND -> G
- C6 pad 2: GND -> G
- C8 pad 1: Net-(C8-Pad1) -> G
- C9 pad 2: Net-(C8-Pad1) -> G
- CON1 pad 2: GND -> G
- CON1 pad 3: GND -> G
- DS1 pad 2: 5V_POWER -> conn_VCC
- IC1 pad 17: BUZZ_control -> Net-(IC1-Pad17)
- IC1 pad 23: DHT11_DATA -> Net-(IC1-Pad23)
- IC1 pad 27: DS1307_SDA -> Net-(IC1-Pad27)
- IC1 pad 28: DS1307_SCL -> Net-(IC1-Pad28)
- IC1 pad 7: 5V_POWER -> conn_VCC
- L1 pad 1: 5V_POWER -> conn_VCC
- P1 pad 1: Net-(C8-Pad1) -> G
- P2 pad 4: GND -> G
- R1 pad 1: 5V_POWER -> conn_VCC
- R3 pad 1: 5V_POWER -> conn_VCC
- R6 pad 1: 5V_POWER -> conn_VCC
- RN1 pad 1: 5V_POWER -> conn_VCC
- U1 pad 4: Net-(C8-Pad1) -> G

Commit message: PCB Design Ver.1.0Beta
PCB Design Ver.1.0Beta
Parts:
- removed C13: 0.1u, Capacitors_SMD:C_1812_HandSoldering
- removed DS1: RC1602A-GHW-ESX, Pin_Headers:Pin_Header_Straight_1x16_Pitch2.54mm
- removed P3: POWER_CONN, Pin_Headers:Pin_Header_Straight_2x01_Pitch2.54mm
- removed RN1: 10K, Pin_Headers:Pin_Header_Straight_1x05_Pitch2.54mm
- added P10: DHT11_conn_B, Pin_Headers:Pin_Header_Straight_1x04_Pitch2.54mm, F.Cu at (44.0, 138.0)
- added P11: DHT11_conn_A, Pin_Headers:Pin_Header_Straight_1x04_Pitch2.54mm, F.Cu at (57.2, 32.2)
- added P7: LCM_D, Pin_Headers:Pin_Header_Straight_1x06_Pitch2.54mm, F.Cu at (73.0, 140.0)
- added P8: DS1307_conn_A, Pin_Headers:Pin_Header_Straight_1x04_Pitch2.54mm, F.Cu at (41.2, 32.2)
- added P9: DS1307_conn_B, Pin_Headers:Pin_Header_Straight_1x04_Pitch2.54mm, F.Cu at (51.2, 177.8)
- added R10: 10k, Resistors_ThroughHole:R_Axial_DIN0207_L6.3mm_D2.5mm_P10.16mm_Horizontal, F.Cu at (77.2, 134.8)
- added R11: 10k, Resistors_ThroughHole:R_Axial_DIN0207_L6.3mm_D2.5mm_P10.16mm_Horizontal, F.Cu at (77.2, 132.5)
- added R12: 10k, Resistors_ThroughHole:R_Axial_DIN0207_L6.3mm_D2.5mm_P10.16mm_Horizontal, F.Cu at (80.5, 132.5)
- added R9: 10k, Resistors_ThroughHole:R_Axial_DIN0207_L6.3mm_D2.5mm_P10.16mm_Horizontal, F.Cu at (80.5, 134.8)
- C1: footprint Capacitors_Tantalum_SMD:CP_Tantalum_Case-D_EIA-7343-31_Wave -> Capacitors_ThroughHole:CP_Radial_D5.0mm_P2.50mm
- C10, C6, C7, C8, C9: footprint Capacitors_SMD:C_1812_HandSoldering -> Capacitors_ThroughHole:C_Disc_D5.0mm_W2.5mm_P5.00mm
- C11, C12: footprint Capacitors_SMD:C_0805_HandSoldering -> Capacitors_ThroughHole:C_Disc_D3.0mm_W1.6mm_P2.50mm
- C2: footprint Capacitors_Tantalum_SMD:CP_Tantalum_Case-X_EIA-7343-43_Wave -> Capacitors_ThroughHole:C_Disc_D5.0mm_W2.5mm_P5.00mm
- C3, C4: footprint Capacitors_SMD:C_1812_HandSoldering -> Capacitors_ThroughHole:C_Disc_D4.7mm_W2.5mm_P5.00mm
- C5: footprint Capacitors_SMD:CP_Elec_4x5.7 -> Capacitors_ThroughHole:CP_Radial_D5.0mm_P2.50mm
- P1: footprint Sockets_WAGO734:WAGO_734_2pin_Straight_RuggedPads -> Socket_Strips:Socket_Strip_Straight_2x01_Pitch2.54mm
- P4: value POWER_CONN -> SW_Part_B; footprint Pin_Headers:Pin_Header_Straight_2x01_Pitch2.54mm -> Pin_Headers:Pin_Header_Straight_1x05_Pitch2.54mm
- P5: value CONN_01X05 -> SW_Part_A
- P6: value CONN_01X05 -> LCM_P; footprint Pin_Headers:Pin_Header_Straight_1x05_Pitch2.54mm -> Pin_Headers:Pin_Header_Straight_1x06_Pitch2.54mm
- Q1, Q2: footprint TO_SOT_Packages_SMD:SOT89-3_Housing_Handsoldering -> TO_SOT_Packages_THT:TO-92_Inline_Wide
- SW1, SW2, SW3, SW4: footprint Buttons_Switches_ThroughHole:SW_Tactile_SKHH_Angled -> Buttons_Switches_ThroughHole:SW_PUSH_SMALL
- moved R8 257.6 mm to (45.0, 17.8), turned to 270 degrees
- moved SW3 247.9 mm to (23.8, 49.5), turned to 0 degrees
- moved SW4 239.2 mm to (23.8, 79.6), turned to 0 degrees
- moved R4 220.3 mm to (67.2, 27.8), turned to 90 degrees
- moved L1 219.6 mm to (52.0, 138.0), turned to 270 degrees
- moved R7 216.6 mm to (48.2, 17.8), turned to 270 degrees
- moved D1 215.6 mm to (60.8, 111.5)
- moved R2 215.6 mm to (54.8, 133.2), turned to 0 degrees
- moved C4 214.8 mm to (48.5, 150.8), turned to 270 degrees
- moved R3 214.5 mm to (54.8, 130.0), turned to 0 degrees
- moved C7 214.0 mm to (52.0, 150.8), turned to 270 degrees
- moved R5 210.2 mm to (58.8, 116.8), turned to 270 degrees
- moved Q2 210.0 mm to (65.5, 119.2)
- moved BZ1 206.8 mm to (76.8, 114.0), turned to 180 degrees
- moved Q1 200.5 mm to (67.5, 125.2), turned to 180 degrees
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Connections:
- BZ1 pad 1: conn_VCC -> 5V_POWER
- C10 pad 1: 5V_POWER -> DHT11_Power
- C10 pad 2: G -> G2
- C2 pad 2: conn_VCC -> 5V_POWER
- C5 pad 2: G -> GND
- C6 pad 2: G -> GND
- C8 pad 1: G -> G1
- C9 pad 1: 5V_POWER -> DS1307_Power
- C9 pad 2: G -> G1
- CON1 pad 2: G -> GND
- CON1 pad 3: G -> GND
- IC1 pad 11: LCM_E -> LCM_D4
- IC1 pad 12: LCM_D4 -> LCM_D5
- IC1 pad 13: LCM_D5 -> LCM_D6
- IC1 pad 14: LCM_D6 -> LCM_D7
- IC1 pad 15: LCM_D7 -> BL
- IC1 pad 16: BL -> Net-(IC1-Pad16)
- IC1 pad 17: Net-(IC1-Pad17) -> BUZZ_control
- IC1 pad 23: Net-(IC1-Pad23) -> func_DOWN
- IC1 pad 24: func_UP -> Menu/Enter
- IC1 pad 25: func_DOWN -> func_UP
- IC1 pad 26: Menu/Enter -> Back/Alarm
- IC1 pad 4: Back/Alarm -> Vo
- IC1 pad 5: Vo -> LCM_RS
- IC1 pad 6: LCM_RS -> LCM_E
- IC1 pad 7: conn_VCC -> 5V_POWER
- L1 pad 1: conn_VCC -> 5V_POWER
- P1 pad 1: G -> Net-(C8-Pad2)
- P1 pad 2: Net-(C8-Pad2) -> G1
- P2 pad 1: 5V_POWER -> DHT11_Power
- P2 pad 4: G -> G2
- P4 pad 1: 5V_POWER -> Net-(P4-Pad1)
- P4 pad 2: G -> Net-(P4-Pad2)
- P5 pad 1: G -> Back/Alarm
- P5 pad 2: BUZZ_control -> func_UP
- P5 pad 3: DS1307_SCL -> Menu/Enter
- P5 pad 4: DS1307_SDA -> func_DOWN
- P5 pad 5: DHT11_DATA -> GND
- P6 pad 1: Net-(IC1-Pad17) -> GND
- P6 pad 2: Net-(IC1-Pad23) -> 5V_POWER
- P6 pad 3: Net-(IC1-Pad27) -> Vo
- P6 pad 4: Net-(IC1-Pad28) -> LCM_RS
- R1 pad 1: conn_VCC -> 5V_POWER
- R3 pad 1: conn_VCC -> 5V_POWER
- R4 pad 2: 5V_POWER -> DHT11_Power
- R6 pad 1: conn_VCC -> 5V_POWER
- R7 pad 1: 5V_POWER -> DS1307_Power
- R8 pad 1: 5V_POWER -> DS1307_Power
- SW1 pad 1: func_UP -> Net-(P4-Pad5)
- SW1 pad 2: GND -> Net-(P4-Pad2)
- SW2 pad 1: func_DOWN -> Net-(P4-Pad4)
- SW2 pad 2: GND -> Net-(P4-Pad5)
- SW3 pad 1: Back/Alarm -> Net-(P4-Pad1)
- SW3 pad 2: GND -> Net-(P4-Pad5)
- SW4 pad 1: Menu/Enter -> Net-(P4-Pad3)
- SW4 pad 2: GND -> Net-(P4-Pad5)
- U1 pad 4: G -> G1
- U1 pad 8: 5V_POWER -> DS1307_Power
Routing:
- net 5V_POWER: track 0.00 -> 307.5 mm
- net GND: track 0.00 -> 206.2 mm
- net Net-(P4-Pad5): track 0.00 -> 90.4 mm
- net Net-(P4-Pad1): track 0.00 -> 37.6 mm
- net DS1307_Power: track 0.00 -> 35.0 mm
- net DHT11_Power: track 0.00 -> 25.6 mm
- net DS1307_SCL: track 0.00 -> 25.2 mm
- net DHT11_DATA: track 0.00 -> 24.8 mm
- net LCM_D4: track 0.00 -> 24.5 mm
- net Menu/Enter: track 0.00 -> 23.0 mm
- net LCM_D7: track 0.00 -> 22.0 mm
- net G1: track 0.00 -> 20.4 mm
- net Net-(P4-Pad4): track 0.00 -> 19.3 mm
- net LCM_D5: track 0.00 -> 18.8 mm
- net LCM_D6: track 0.00 -> 18.4 mm
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- added copper zone on B.Cu, net G1
- added copper zone on B.Cu, net G2
- added copper zone on B.Cu, net Net-(P4-Pad5)
Other:
- net class Default: trace_width 0.25 -> 0.8

Commit message: PCB Design V1.2
PCB Design V1.2
Parts:
- added REF**: MountingHole_3.5mm_Pad_Via, Mounting_Holes:MountingHole_3.5mm_Pad_Via, F.Cu at (76.0, 112.0)
- added REF**: MountingHole_3.5mm_Pad_Via, Mounting_Holes:MountingHole_3.5mm_Pad_Via, F.Cu at (25.0, 112.0)
- added REF**: MountingHole_3.5mm_Pad_Via, Mounting_Holes:MountingHole_3.5mm_Pad_Via, F.Cu at (76.0, 53.0)
- added REF**: MountingHole_3.5mm_Pad_Via, Mounting_Holes:MountingHole_3.5mm_Pad_Via, F.Cu at (25.0, 53.0)
- added REF**: MountingHole_3.5mm_Pad_Via, Mounting_Holes:MountingHole_3.5mm_Pad_Via, F.Cu at (95.0, 38.0)
- added REF**: MountingHole_3.5mm_Pad_Via, Mounting_Holes:MountingHole_3.5mm_Pad_Via, F.Cu at (95.0, 78.0)
- moved P4 74.0 mm to (104.0, 51.0)
- moved SW1 74.0 mm to (94.8, 48.5)
- moved SW2 74.0 mm to (94.8, 68.8)
- moved SW3 74.0 mm to (94.8, 28.5)
- moved SW4 74.0 mm to (94.8, 58.6)
- moved BZ1 66.9 mm to (65.8, 48.0)
- moved C1 66.9 mm to (67.0, 98.8)
- moved C11 66.9 mm to (62.0, 87.2)
- moved C12 66.9 mm to (62.0, 79.8)
- moved C2 66.9 mm to (58.0, 106.2)
- moved C3 66.9 mm to (52.5, 107.0)
- moved C4 66.9 mm to (37.5, 84.8)
- moved C5 66.9 mm to (34.7, 54.8)
- moved C6 66.9 mm to (43.4, 53.0)
- moved C7 66.9 mm to (41.0, 84.8)
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Routing:
- added copper zone on B.Cu, net GND
